Commit message: fix

File: urdf/whill.urdf (robot description, URDF)
Before this commit: robot whill_urdf, 5 links, 4 joints
Links:
- link base_link: geometry collision mesh filename=package://whill_description/meshes/base_link.stl scale=0.001 0.001 0.001; visual mesh filename=package://whill_description/meshes/base_link.stl scale=0.001 0.001 0.001

Commit message: fix velodyne frame

File: urdf/whill.urdf (robot description, URDF)
Before this commit: robot whill_urdf, 5 links, 4 joints
Links:
- removed link velodyne_link
- added link velodyne
Joints:
- joint velodyne_joint: child velodyne_link -> velodyne

Commit message: update

File: urdf/whill.urdf (robot description, URDF)
Before this commit: robot whill_urdf, 5 links, 4 joints
Links:
- added link camera_link
Joints:
- added joint camera_joint: type fixed, parent base_link, child camera_link, origin xyz=0.265214 0.011291 0.963493 rpy=0 0 0
- joint center_mid_joint: origin xyz=0.234214 0.011291 0.867876 rpy=3.1416 -0.0349 0 -> xyz=0.234214 0.011291 0.867876 rpy=3.1416 -0.0349 0.0
- joint left_mid_joint: origin xyz=0.235214 0.273508 0.823493 rpy=-1.5708 -1.6057 0 -> xyz=0.235214 0.273508 0.867876 rpy=-1.5708 -1.6057 0
- joint right_mid_joint: origin xyz=0.234214 -0.274326 0.823493 rpy=1.5708 -1.6057 0 -> xyz=0.234214 -0.274326 0.867876 rpy=1.5708 -1.6057 0
- joint velodyne_joint: origin xyz=0.177514 0.009591 1.384793 rpy=0 0.0349 0 -> xyz=0.177514 0.009591 1.384793 rpy=0 0.0349 -0.035266462599716
